File: Preselector.brd (EAGLE design)
At the start: 183 x 123.8 mm, 167 parts, among them IC4 TPS7A8101DRB, IC58 LMZ31707RVQ, Q2 FDV303N, X1 0733660061, X10 0733660061, X11 0733660061, X12 0733660061, X13 0733660061, X14 0733660061, X15 0733660061, X16 0733660061, X17 0733660061, X18 0733660061, X19 0733660061, X2 0733660061, X20 0733660061, X21 0733660061, X22 0733660061, X23 0733660061, X24 0733660061, X25 0733660061, X26 0733660061, X27 0733660061, X28 0733660061, X29 0733660061, X3 0733660061, X30 0733660061, X31 0733660061, X32 0733660061, X4 0733660061, X5 0733660061, X6 0733660061, X7 0733660061, X8 0733660061, X9 0733660061

Commit message: Routed all signal wires, left notes on the board for you. Next we need  to add an LDO to each amplifier on the schematic. Will be quite a bit of work. All traces on the schematic have been renamed properly.
Parts:
- moved L1 5.11 mm to (52.8, 55.5)
- moved C3 4.85 mm to (50.3, 58.3)
- moved C2 4.83 mm to (47.9, 58.3)
- moved L2 4.75 mm to (56.8, 56.9), turned to 270 degrees
- moved C1 4.38 mm to (48.4, 55.0), turned to 0 degrees
- moved C4 4.34 mm to (55.8, 52.1)
- moved LNA_1 3.82 mm to (50.2, 52.3)
- moved L26 3.70 mm to (156.1, 11.0)
- moved C42 2.34 mm to (51.2, 8.51), turned to 90 degrees
- moved C46 2.30 mm to (92.3, 8.51), turned to 90 degrees
- moved C50 2.29 mm to (133.7, 8.51), turned to 90 degrees
- moved L16 2.09 mm to (15.4, 8.76)
- moved L23 1.48 mm to (123.1, 5.21)
- moved L20 1.08 mm to (81.9, 5.21)
- moved L21 1.05 mm to (90.0, 11.8)
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Routing:
- net SAW_15_IN: track 0.00 -> 19.8 mm
- net SAW_14_IN: track 0.00 -> 19.4 mm
- net SAW_16_IN: track 0.21 -> 19.2 mm
- net SAW_1_OUT: track 0.00 -> 17.9 mm
- net SAW_13_OUT: track 0.00 -> 17.4 mm
- net SAW_3_OUT: track 0.00 -> 17.4 mm
- net SAW_4_IN: track 0.36 -> 17.7 mm
- net SAW_2_IN: track 0.00 -> 17.0 mm
- net SAW_15_OUT: track 0.00 -> 16.9 mm
- net SAW_14_OUT: track 0.00 -> 16.6 mm
- net SAW_3_IN: track 0.54 -> 16.8 mm
- net SAW_6_IN: track 0.00 -> 15.2 mm
- net SAW_7_IN: track 0.00 -> 15.0 mm
- net SAW_2_OUT: track 0.00 -> 14.9 mm
- net SAW_5_IN: track 0.00 -> 14.2 mm
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- added copper zone on layer 1, net D'GND
- added copper zone on layer 1, net N$7
Other:
- board text added: "This ground needs to be up like the 4m and 2m for all these style caps. Via should be 3 grid spaces away at 10mil, if no room then 2 is fine."
- board text added: "You must do a "poly 'gnd" each polygon to associate it with ground."
- board text added: "You must do a "via 'gnd" command to make the via a ground otherwise you will see circles in the polygon"
- board text removed: "Aligned"
- board text removed: "Misaligned by 5mil"
