File: Preselector - Copy.brd (EAGLE design)
At the start: 160 x 100 mm, 120 parts, among them IC58 LMZ31707RVQ, Q2 FDV303N, X1 0733660061, X2 0733660061, X3 0733660061, X4 0733660061, X5 0733660061, X6 0733660061

Commit message: All components should be connected to ground as well as all pre_pwr wires have been routed. 4 air wires remain...
Parts:
- removed L47: 56n 1206, NewSDR:C1206
- removed U$1, U$2, U$3, U$4: TA1914A, SeniorDesign:TA1914A
- added C100, C101, C53, C54, C58, C59, C62, C63, C66, C67, C70, C71, C76, C77, C80, C81, C84, C85, C88, C89, C92, C93, C96, C97: 470n, rcl:C0402K
- added C102, C103, C55, C56, C60, C61, C64, C65, C68, C69, C74, C75, C78, C79, C82, C83, C86, C87, C90, C91, C94, C95, C98, C99: NFM21PS106B0J3D, DEEP EDDY:NFM21PS
- added C50: 160p, rcl:C0603K
- added C51: 180p, rcl:C0603K
- added L23, L24, L25, L26: 100n, NewSDR:C1206
- added LDO_1, LDO_10, LDO_11, LDO_12, LDO_2, LDO_3, LDO_4, LDO_5, LDO_6, LDO_7, LDO_8, LDO_9: TPS7A8101DRB, DEEP EDDY:DRB
- added LNA_10, LNA_11, LNA_12: SPF-5043Z, SeniorDesign:SPF-5043Z
- added R1, R10, R11, R14, R15, R19, R21, R23, R24, R26, R27, R29, R3, R30, R32, R33, R35, R36, R38, R39, R41, R5, R7, R8: 10.0k, rcl:R0603
- added R12, R16, R2, R22, R25, R28, R31, R34, R37, R40, R6, R9: 52.3k, rcl:R0603
- added SAW_10, SAW_11, SAW_12, SAW_9: TA1914A, SeniorDesign:TA1914A
- added SAW_13, SAW_14, SAW_15, SAW_16: S511214, SeniorDesign:S511214
- added TP_1, TP_10, TP_11, TP_12, TP_2, TP_3, TP_4, TP_5, TP_6, TP_7, TP_8, TP_9: TPTP20SQ, testpad:TP20SQ
- added X10, X11, X12, X13, X14, X15, X16, X17, X18, X19, X20, X21, X22, X23, X24, X25, X26, X27, X28, X29, X30, X31, X32, X7, X8, X9: 0733660061, con-coax:BU-SMA-V
- C1, C11, C18, C20, C22, C24, C26, C28, C3, C30, C32, C36, C37: value 100p 50v c0g -> 100p
- C10: value 0.1u 16V X7R -> 0.1u
- C12, C8: value 100p 50v c0g -> 8p
- C13: value 0.1u 16V X7R -> 12p
- C14, C16: value 8p 5% 0603 -> 100p
- C15: value 12p 5% 0603 -> 0.1u
- C17, C7: value 12p 5% 0603 -> 100p
- C19, C2, C23, C27, C31, C44: value 100p 50v c0g -> 0.1u
- C21, C25, C29, C33, C45: value 0.1u 16V X7R -> 100p
- C34, C41, C49: value 2pF -> 100p
- C35, C40, C48: value 2pF -> 0.1u
- C38, C42: value 100p 50v c0g -> 160p
- C39: value 0.1u 16V X7R -> 180p
- C4: value 0.1u 16V X7R -> 8p
- C43: value 100p 50v c0g -> 180p
- C46: value 2pF -> 160p
- C47: value 2pF -> 180p
- C5, C9: value 100p 50v c0g -> 12p
- C6: value 8p 5% 0603 -> 0.1u
- L1: value 47n 1206 -> 100n
- L10, L13, L16, L18: value 86n 1206 -> 100n
- L11, L14, L17, L19: value 84n 1206 -> 100n
- L12, L15, L20, L21, L22, L7: value 100n 1206 -> 100n
- L2: value 56n 1206 -> 56n
- L3: value 47n 1206 -> 47n
- L4: value 56n 1206 -> 100n
- L5: value 47n 1206 -> 56n
- L6, L9: value 100n 1206 -> 47n
- L8: value 100n 1206 -> 56n
- TP10: value TPSQTP20SQD -> TPSQB1,27; device testpad:TP20SQD -> testpad:B1,27
- moved R201 274.1 mm to (175.3, 109.2), turned to 180 degrees
- moved R206 255.3 mm to (159.5, 123.7)
- moved C459 254.5 mm to (167.8, 111.3), turned to 270 degrees
- moved LED1 253.2 mm to (178.3, 110.2)
- moved Q2 244.0 mm to (160.0, 117.3), turned to 90 degrees
- moved C13 242.1 mm to (167.6, 49.9)
- moved IC58 238.3 mm to (167.9, 120.7), turned to 90 degrees
- moved SAW_8 236.8 mm to (136.1, 82.6)
- moved C483 230.9 mm to (165.6, 131.6), turned to 270 degrees
- moved C484 227.8 mm to (151.9, 125.5), turned to 90 degrees
- moved C493 227.0 mm to (169.7, 127.5), turned to 180 degrees
- moved C12 226.7 mm to (141.5, 46.7)
- moved C492 226.5 mm to (175.8, 125.0)
- moved TP10 225.1 mm to (176.3, 119.9)
- moved C49 224.4 mm to (127.6, 18.0), turned to 90 degrees
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Connections:
- net N$1 renamed LNA_2_IN
- removed net 1.25M_RF_IN1: C26.2, LNA_6.3
- removed net 1.25M_RF_IN2: C31.2, C34.2
- removed net 1.25M_RF_IN3: C22.1, C22.2, LNA_5.3, SAW_5.6
- removed net 1.25M_RF_IN4: C37.2, C40.2
- removed net 1.25M_RF_IN5: C43.2, C46.2
- removed net 1.25M_RF_IN_: C23.2, SAW_6.2
- removed net 1.25M_RF_IN_1: C27.2, SAW_7.2
- removed net 1.2M5_RF_IN4: C26.1, SAW_6.6
- removed net 2M_RF_IN1: X2.1
- removed net 2M_RF_IN10: C48.1, L18.1
- removed net 2M_RF_IN11: C49.2, X6.1
- removed net 2M_RF_IN2: C18.1, C18.2, LNA_4.3, X3.1
- removed net 2M_RF_IN3: SAW_8.6, X4.1
- removed net 2M_RF_IN4: C30.1, C30.2, LNA_7.3, X5.1
- removed net 2M_RF_IN5: C34.1, L10.1
- removed net 2M_RF_IN6: C36.2, LNA_8.3
- removed net 2M_RF_IN7: C40.1, L13.1
- removed net 2M_RF_IN8: C41.2, C42.1, C42.2, LNA_9.3
- removed net 2M_RF_IN9: C46.1, L16.1
- removed net GND1: C23.1, L6.1, LNA_5.1
- removed net GND2: C19.1, L7.1, LNA_4.1
- removed net GND3: L8.1
- removed net GND4: C31.1, L9.1, LNA_7.1
- removed net GND5: C37.1, L12.1, LNA_8.1
- removed net GND6: C43.1, L15.1, LNA_9.1
- removed net N$10: C15.2, C16.1
- removed net N$11: C16.2, L4.2, SAW_4.2
- removed net N$2: C6.2, L47.2, SAW_2.2
- removed net N$21: C47.1, L17.2
- removed net N$23: L16.2
- removed net N$26: L18.2
- removed net N$29: C35.2, C36.1
- removed net N$3: C14.2, L2.2, SAW_3.2
- removed net N$31: C8.1, L22.2, LNA_3.1
- removed net N$4: C14.1, C8.2
- removed net N$5: C7.1, L1.2, SAW_2.6
- removed net N$6: C11.2, LNA_3.3
- removed net N$7: SAW_2.1, SAW_2.3, SAW_2.4, SAW_2.5, SAW_2.7, SAW_2.8
- removed net N$8: C7.2
- removed net N$9: C15.1, L3.2, SAW_3.6
- new net 1.25_RF_OUT: SAW_8.6, X16.1
- new net 2M_RF_OUT: C13.2, X8.1
- new net 4M_RF_IN: C38.1, L16.1, X25.1
- new net 4M_RF_OUT: C51.2, L26.1, X32.1
- new net 70CM_RF_IN: C26.1, X17.1
- new net 70CM_RF_OUT: SAW_12.5, X24.1
- new net LDO_10_5V: C40.1, C41.1, C93.2, C95.OUT, L18.2, R34.1, TP_10.TP
- new net LDO_11_5V: C44.1, C45.1, C97.2, C99.OUT, L21.2, R37.1, TP_11.TP
- new net LDO_12_5V: C101.2, C103.OUT, C48.1, C49.1, L24.2, R40.1, TP_12.TP
- new net LDO_1_5V: C2.1, C3.1, C54.2, C56.OUT, L1.2, R2.1, TP_1.TP
- new net LDO_2_5V: C59.2, C6.1, C61.OUT, C7.1, L4.2, R6.1, TP_2.TP
- new net LDO_3_5V: C10.1, C11.1, C63.2, C65.OUT, L7.1, R9.1, TP_3.TP
- new net LDO_4_5V: C15.1, C16.1, C67.2, C69.OUT, L10.2, R12.1, TP_4.TP
- new net LDO_5_5V: C19.1, C20.1, C71.2, C75.OUT, L11.2, R16.1, TP_5.TP
- new net LDO_6_5V: C23.1, C24.1, C77.2, C79.OUT, L12.1, R22.1, TP_6.TP
- new net LDO_7_5V: C27.1, C28.1, C81.2, C83.OUT, L13.2, R25.1, TP_7.TP
- new net LDO_8_5V: C31.1, C32.1, C85.2, C87.OUT, L14.2, R28.1, TP_8.TP
- new net LDO_9_5V: C35.1, C36.1, C89.2, C91.OUT, L15.2, R31.1, TP_9.TP
- new net LNA_10_IN: C39.2, L17.1, LNA_10.3
- new net LNA_10_OUT: C42.1, L18.1, L19.1, LNA_10.1
- new net LNA_11_IN: C43.2, L20.1, LNA_11.3
- new net LNA_11_OUT: C46.1, L21.1, L22.1, LNA_11.1
- new net LNA_12_IN: C47.2, L23.1, LNA_12.3
- new net LNA_12_OUT: C50.1, L24.1, L25.1, LNA_12.1
- new net LNA_1_IN: C1.2, LNA_1.3
- new net LNA_1_OUT: C4.1, L1.1, LNA_1.1
- new net LNA_2_OUT: C8.2, L4.1, LNA_2.1
- new net LNA_3_IN: C9.2, LNA_3.3
- new net LNA_3_OUT: C12.1, L7.2, LNA_3.1
- new net LNA_4_IN: C14.2, LNA_4.3
- new net LNA_4_OUT: C17.1, L10.1, LNA_4.1
- new net LNA_5_IN: C18.2, LNA_5.3
- new net LNA_5_OUT: C21.1, L11.1, LNA_5.1
- new net LNA_6_IN: C22.2, LNA_6.3
- new net LNA_6_OUT: C25.1, L12.2, LNA_6.1
- new net LNA_7_IN: C26.2, LNA_7.3
- new net LNA_7_OUT: C29.1, L13.1, LNA_7.1
- new net LNA_8_IN: C30.2, LNA_8.3
- new net LNA_8_OUT: C33.1, L14.1, LNA_8.1
- new net LNA_9_IN: C34.2, LNA_9.3
- new net LNA_9_OUT: C37.1, L15.1, LNA_9.1
- new net N$33: C69.IN, LDO_4.1, LDO_4.2
- new net N$34: C71.1, LDO_5.3, R16.2, R19.1
- new net N$36: C70.1, LDO_5.6
- new net N$38: C74.OUT, LDO_5.7, LDO_5.8
- new net N$39: C75.IN, LDO_5.1, LDO_5.2
- new net N$40: C81.1, LDO_7.3, R25.2, R26.1
- new net N$41: C77.1, LDO_6.3, R22.2, R23.1
- new net N$42: C76.1, LDO_6.6
- new net N$43: C78.OUT, LDO_6.7, LDO_6.8
- new net N$45: C79.IN, LDO_6.1, LDO_6.2
- new net N$46: C80.1, LDO_7.6
- new net N$47: C82.OUT, LDO_7.7, LDO_7.8
- new net N$48: C83.IN, LDO_7.1, LDO_7.2
- new net N$49: C85.1, LDO_8.3, R28.2, R29.1
- new net N$50: C84.1, LDO_8.6
- new net N$51: C86.OUT, LDO_8.7, LDO_8.8
- new net N$52: C87.IN, LDO_8.1, LDO_8.2
- new net N$53: C89.1, LDO_9.3, R31.2, R32.1
- new net N$54: C88.1, LDO_9.6
- new net N$56: C90.OUT, LDO_9.7, LDO_9.8
- new net N$57: C91.IN, LDO_9.1, LDO_9.2
- new net N$61: C93.1, LDO_10.3, R34.2, R35.1
- new net N$62: C92.1, LDO_10.6
- new net N$63: C94.OUT, LDO_10.7, LDO_10.8
- new net N$64: C95.IN, LDO_10.1, LDO_10.2
- new net N$66: C97.1, LDO_11.3, R37.2, R38.1
- new net N$67: C96.1, LDO_11.6
- new net N$68: C98.OUT, LDO_11.7, LDO_11.8
- new net N$69: C99.IN, LDO_11.1, LDO_11.2
- new net N$70: C101.1, LDO_12.3, R40.2, R41.1
- new net N$71: C100.1, LDO_12.6
- new net N$72: C102.OUT, LDO_12.7, LDO_12.8
- new net N$73: C103.IN, LDO_12.1, LDO_12.2
- new net PRE_PWR_10: LDO_1.5, LDO_10.5, LDO_11.5, LDO_2.5, LDO_3.5, LDO_4.5, LDO_5.5, LDO_6.5, LDO_7.5, LDO_8.5, LDO_9.5, R1.2, R11.2, R15.2, R21.2, R24.2, R27.2, R30.2, R33.2, R36.2, R5.2, R8.2
- new net PRE_PWR_12: LDO_12.5, R39.2
- new net SAW+6_OUT: C22.1, SAW_6.6, X13.1
- new net SAW_10_IN: C33.2, SAW_10.2, X20.1
- new net SAW_10_OUT: C34.1, SAW_10.5, X21.1
- new net SAW_11_12_RF: SAW_11.5, SAW_12.2, X23.1
- new net SAW_11_IN: C37.2, SAW_11.2, X22.1
- new net SAW_13_IN: C38.2, SAW_13.10
- new net SAW_13_OUT: C39.1, SAW_13.5, X26.1
- new net SAW_14_IN: C42.2, SAW_14.10, X27.1
- new net SAW_14_OUT: C43.1, SAW_14.5, X28.1
- new net SAW_15_IN: C46.2, SAW_15.10, X29.1
- new net SAW_15_OUT: C47.1, SAW_15.5, X30.1
- new net SAW_16_IN: C50.2, SAW_16.10, X31.1
- new net SAW_16_OUT: C51.1, SAW_16.5
- new net SAW_1_OUT: C1.1, SAW_1.8, X2.1
- new net SAW_2_IN: C4.2, L2.2, SAW_2.2, X3.1
- new net SAW_2_OUT: C5.1, L3.2, SAW_2.6, X4.1
- new net SAW_3_IN: C8.1, L5.2, SAW_3.2, X5.1
- new net SAW_3_OUT: C9.1, L6.2, SAW_3.6, X6.1
- new net SAW_4_IN: C12.2, L8.2, SAW_4.2, X7.1
- new net SAW_4_OUT: C13.1, L9.2, SAW_4.6
- new net SAW_5_IN: C17.2, SAW_5.2, X10.1
- new net SAW_5_OUT: C18.1, SAW_5.6, X11.1
- new net SAW_6_IN: C21.2, SAW_6.2, X12.1
- new net SAW_7_8_RF: SAW_7.6, SAW_8.2, X15.1
- new net SAW_7_IN: C25.2, SAW_7.2, X14.1
- new net SAW_9_IN: C29.2, SAW_9.2, X18.1
- new net SAW_9_OUT: C30.1, SAW_9.5, X19.1
- net +5V3: now also C102.IN, C55.IN, C60.IN, C64.IN, C68.IN, C74.IN, C78.IN, C82.IN, C86.IN, C90.IN, C94.IN, C98.IN, R1.1, R11.1, R15.1, R21.1, R24.1, R27.1, R30.1, R33.1, R36.1, R39.1, R5.1, R8.1; no longer C10.1, C12.1, C13.1, C20.1, C21.1, C24.1, C25.1, C28.1, C29.1, C3.1, C32.1, C33.1, C38.1, C39.1, C4.1, C44.1, C45.1, C9.1, L12.2, L15.2, L20.2, L21.2, L6.2, L7.2, L9.2
- net 1.25M_RF_IN: now also C14.1, X9.1; no longer C19.2, SAW_5.2
- net 2M_RF_IN: no longer C1.1, C1.2, C2.2, C5.1, LNA_1.3, SAW_1.8
- net GND: now also C100.2, C102.GND1, C102.GND2, C102.GND3, C102.GND4, C102.GND5, C102.GND6, C102.GND7, C102.GND8, C103.GND1, C103.GND2, C103.GND3, C103.GND4, C103.GND5, C103.GND6, C103.GND7, C103.GND8, C11.2, C15.2, C16.2, C19.2, C2.2, C23.2, C27.2, C31.2, C35.2, C36.2, C40.2, C41.2, C48.2, C49.2, C53.2, C55.GND1, C55.GND2, C55.GND3, C55.GND4, C55.GND5, C55.GND6, C55.GND7, C55.GND8, C56.GND1, C56.GND2, C56.GND3, C56.GND4, C56.GND5, C56.GND6, C56.GND7, C56.GND8, C58.2, C6.2, C60.GND1, C60.GND2, C60.GND3, C60.GND4, C60.GND5, C60.GND6, C60.GND7, C60.GND8, C61.GND1, C61.GND2, C61.GND3, C61.GND4, C61.GND5, C61.GND6, C61.GND7, C61.GND8, C62.2, C64.GND1, C64.GND2, C64.GND3, C64.GND4, C64.GND5, C64.GND6, C64.GND7, C64.GND8, C65.GND1, C65.GND2, C65.GND3, C65.GND4, C65.GND5, C65.GND6, C65.GND7, C65.GND8, C66.2, C68.GND1, C68.GND2, C68.GND3, C68.GND4, C68.GND5, C68.GND6, C68.GND7, C68.GND8, C69.GND1, C69.GND2, C69.GND3, C69.GND4, C69.GND5, C69.GND6, C69.GND7, C69.GND8, C7.2, C70.2, C74.GND1, C74.GND2, C74.GND3, C74.GND4, C74.GND5, C74.GND6, C74.GND7, C74.GND8, C75.GND1, C75.GND2, C75.GND3, C75.GND4, C75.GND5, C75.GND6, C75.GND7, C75.GND8, C76.2, C78.GND1, C78.GND2, C78.GND3, C78.GND4, C78.GND5, C78.GND6, C78.GND7, C78.GND8, C79.GND1, C79.GND2, C79.GND3, C79.GND4, C79.GND5, C79.GND6, C79.GND7, C79.GND8, C80.2, C82.GND1, C82.GND2, C82.GND3, C82.GND4, C82.GND5, C82.GND6, C82.GND7, C82.GND8, C83.GND1, C83.GND2, C83.GND3, C83.GND4, C83.GND5, C83.GND6, C83.GND7, C83.GND8, C84.2, C86.GND1, C86.GND2, C86.GND3, C86.GND4, C86.GND5, C86.GND6, C86.GND7, C86.GND8, C87.GND1, C87.GND2, C87.GND3, C87.GND4, C87.GND5, C87.GND6, C87.GND7, C87.GND8, C88.2, C90.GND1, C90.GND2, C90.GND3, C90.GND4, C90.GND5, C90.GND6, C90.GND7, C90.GND8, C91.GND1, C91.GND2, C91.GND3, C91.GND4, C91.GND5, C91.GND6, C91.GND7, C91.GND8, C92.2, C94.GND1, C94.GND2, C94.GND3, C94.GND4, C94.GND5, C94.GND6, C94.GND7, C94.GND8, C95.GND1, C95.GND2, C95.GND3, C95.GND4, C95.GND5, C95.GND6, C95.GND7, C95.GND8, C96.2, C98.GND1, C98.GND2, C98.GND3, C98.GND4, C98.GND5, C98.GND6, C98.GND7, C98.GND8, C99.GND1, C99.GND2, C99.GND3, C99.GND4, C99.GND5, C99.GND6, C99.GND7, C99.GND8, L16.2, L17.2, L19.2, L20.2, L22.2, L23.2, L25.2, L26.2, L6.1, L8.1, L9.1, LDO_1.4, LDO_1.P1, LDO_1.P2, LDO_1.P3, LDO_1.P4, LDO_1.P5, LDO_1.PAD, LDO_10.4, LDO_10.P1, LDO_10.P2, LDO_10.P3, LDO_10.P4, LDO_10.P5, LDO_10.PAD, LDO_11.4, LDO_11.P1, LDO_11.P2, LDO_11.P3, LDO_11.P4, LDO_11.P5, LDO_11.PAD, LDO_12.4, LDO_12.P1, LDO_12.P2, LDO_12.P3, LDO_12.P4, LDO_12.P5, LDO_12.PAD, LDO_2.4, LDO_2.P1, LDO_2.P2, LDO_2.P3, LDO_2.P4, LDO_2.P5, LDO_2.PAD, LDO_3.4, LDO_3.P1, LDO_3.P2, LDO_3.P3, LDO_3.P4, LDO_3.P5, LDO_3.PAD, LDO_4.4, LDO_4.P1, LDO_4.P2, LDO_4.P3, LDO_4.P4, LDO_4.P5, LDO_4.PAD, LDO_5.4, LDO_5.P1, LDO_5.P2, LDO_5.P3, LDO_5.P4, LDO_5.P5, LDO_5.PAD, LDO_6.4, LDO_6.P1, LDO_6.P2, LDO_6.P3, LDO_6.P4, LDO_6.P5, LDO_6.PAD, LDO_7.4, LDO_7.P1, LDO_7.P2, LDO_7.P3, LDO_7.P4, LDO_7.P5, LDO_7.PAD, LDO_8.4, LDO_8.P1, LDO_8.P2, LDO_8.P3, LDO_8.P4, LDO_8.P5, LDO_8.PAD, LDO_9.4, LDO_9.P1, LDO_9.P2, LDO_9.P3, LDO_9.P4, LDO_9.P5, LDO_9.PAD, LNA_10.2, LNA_10.4, LNA_11.2, LNA_11.4, LNA_12.2, LNA_12.4, R10.2, R14.2, R19.2, R23.2, R26.2, R29.2, R3.2, R32.2, R35.2, R38.2, R41.2, R7.2, SAW_10.1, SAW_10.3, SAW_10.4, SAW_10.6, SAW_11.1, SAW_11.3, SAW_11.4, SAW_11.6, SAW_12.1, SAW_12.3, SAW_12.4, SAW_12.6, SAW_13.1, SAW_13.2, SAW_13.3, SAW_13.4, SAW_13.6, SAW_13.7, SAW_13.8, SAW_13.9, SAW_14.1, SAW_14.2, SAW_14.3, SAW_14.4, SAW_14.6, SAW_14.7, SAW_14.8, SAW_14.9, SAW_15.1, SAW_15.2, SAW_15.3, SAW_15.4, SAW_15.6, SAW_15.7, SAW_15.8, SAW_15.9, SAW_16.1, SAW_16.2, SAW_16.3, SAW_16.4, SAW_16.6, SAW_16.7, SAW_16.8, SAW_16.9, SAW_2.1, SAW_2.3, SAW_2.4, SAW_2.5, SAW_2.7, SAW_2.8, SAW_5.1, SAW_5.3, SAW_5.4, SAW_5.5, SAW_5.7, SAW_5.8, SAW_6.1, SAW_6.3, SAW_6.4, SAW_6.5, SAW_6.7, SAW_6.8, SAW_7.1, SAW_7.3, SAW_7.4, SAW_7.5, SAW_7.7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; no longer C12.2, C13.2, C21.2, C25.2, C29.2, C33.2, C38.2, C39.2, C4.2, C9.2, L1.1, L4.1, L47.1
- net N$12: now also C54.1, LDO_1.3, R2.2, R3.1; no longer C17.1, L5.2, SAW_4.6
- net N$13: now also C53.1, LDO_1.6; no longer C27.1, L8.2, LNA_6.1
- net N$14: now also C55.OUT, LDO_1.7, LDO_1.8; no longer SAW_7.6, SAW_8.2
- net N$15: now also C56.IN, LDO_1.1, LDO_1.2; no longer C35.1, L11.2
- net N$16: now also C59.1, LDO_2.3, R6.2, R7.1; no longer L11.1
- net N$17: now also C58.1, LDO_2.6; no longer L10.2
- net N$18: now also C60.OUT, LDO_2.7, LDO_2.8; no longer C41.1, L14.2
- net N$180: no longer TP10.1
- net N$19: now also C61.IN, LDO_2.1, LDO_2.2; no longer L14.1
- net N$20: now also C63.1, LDO_3.3, R10.1, R9.2; no longer L13.2
- net N$22: now also C62.1, LDO_3.6; no longer L17.1
- net N$24: now also C64.OUT, LDO_3.7, LDO_3.8; no longer C49.1, L19.2
- net N$25: now also C65.IN, LDO_3.1, LDO_3.2; no longer L19.1
- net N$27: now also C67.1, LDO_4.3, R12.2, R14.1; no longer C47.2, C48.2
- net N$28: now also C66.1, LDO_4.6; no longer C6.1, L21.1, LNA_2.1
- net N$30: now also C68.OUT, LDO_4.7, LDO_4.8; no longer C2.1, L20.1, LNA_1.1
Routing:
- net LDO_3_5V: track 0.00 -> 44.7 mm
- net LDO_10_5V: track 0.00 -> 44.7 mm
- net LDO_12_5V: track 0.00 -> 44.7 mm
- net LDO_4_5V: track 0.00 -> 43.7 mm
- net LDO_8_5V: track 0.00 -> 43.6 mm
- net LDO_7_5V: track 0.00 -> 43.5 mm
- net LDO_9_5V: track 0.00 -> 43.1 mm
- net LDO_11_5V: track 0.00 -> 42.7 mm
- net LDO_5_5V: track 0.00 -> 41.0 mm
- net LDO_2_5V: track 0.00 -> 41.0 mm
- net LDO_6_5V: track 0.00 -> 40.2 mm
- net LDO_1_5V: track 0.00 -> 39.8 mm
- net SAW_15_IN: track 0.00 -> 19.6 mm
- net SAW_16_IN: track 0.00 -> 19.2 mm
- net SAW_14_IN: track 0.00 -> 18.8 mm
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- added copper zone on layer 1, net +13.8V_SW_FIL
- added copper zone on layer 1, net +5V3
- added copper zone on layer 15, net +5V3
- added copper zone on layer 1, net GND
- added copper zone on layer 2, net GND
- added copper zone on layer 1, net N$196
- added copper zone on layer 1, net N$199
Other:
- board size 160 x 100 mm -> 183 x 137.8 mm
- board text added: "1.25m"
- board text added: "2m"
- board text added: "4m"
- board text added: "70cm"
- board text added: "You must do a "poly 'gnd" each polygon to associate it with ground."
- board text added: "You must do a "via 'gnd" command to make the via a ground otherwise you will see circles in the polygon"
