File: Preselector - Copy.sch (EAGLE design)
At the start: 75 parts, among them IC58 LMZ31707RVQ, Q2 FDV303N, X1 0733660061, X2 0733660061, X3 0733660061

Commit message: Saved Preselector to backup
Parts:
- removed IC1, IC2, IC3: (no value), analog-devices:AD102
- added C30, C31, C32, C36, C37, C38, C42, C43, C44: 100p 50v c0g, rcl:C-USC0603K
- added C33, C39, C45: 0.1u 16V X7R, rcl:C-USC0603K
- added C34, C35, C40, C41, C46, C47, C48, C49: 2pF, rcl:C-USC0603K
- added L10, L13, L16, L18: 86n 1206, NewSDR:L-US1206
- added L11, L14, L17, L19: 84n 1206, NewSDR:L-US1206
- added L12, L15, L20, L21, L22, L6, L7, L8, L9: 100n 1206, NewSDR:L-US1206
- added LNA_7, LNA_8, LNA_9: SPF-5043Z, SeniorDesign:SPF-5043Z
- added SAW_8: TA0576A, SeniorDesign:TA0576A
- added U$1, U$2, U$3, U$4: TA1914A, SeniorDesign:TA1914A
- added X4, X5, X6: 0733660061, con-coax:BU-SMA-V
Connections:
- new net 1.25M_RF_IN2: C31.2, C34.2
- new net 1.25M_RF_IN4: C37.2, C40.2
- new net 1.25M_RF_IN5: C43.2, C46.2
- new net 2M_RF_IN10: C48.1, L18.1
- new net 2M_RF_IN11: C49.2, X6G$1.1
- new net 2M_RF_IN3: SAW_8.OUTPUT, X4G$1.1
- new net 2M_RF_IN4: C30.1, C30.2, LNA_7.RF_IN, X5G$1.1
- new net 2M_RF_IN5: C34.1, L10.1
- new net 2M_RF_IN6: C36.2, LNA_8.RF_IN
- new net 2M_RF_IN7: C40.1, L13.1
- new net 2M_RF_IN8: C41.2, C42.1, C42.2, LNA_9.RF_IN
- new net 2M_RF_IN9: C46.1, L16.1
- new net GND1: C23.1, L6.1, LNA_5.RF_OUT
- new net GND2: C19.1, L7.1, LNA_4.RF_OUT
- new net GND3: L8.1
- new net GND4: C31.1, L9.1, LNA_7.RF_OUT
- new net GND5: C37.1, L12.1, LNA_8.RF_OUT
- new net GND6: C43.1, L15.1, LNA_9.RF_OUT
- new net N$13: C27.1, L8.2, LNA_6.RF_OUT
- new net N$14: SAW_7.OUTPUT, SAW_8.INPUT
- new net N$15: C35.1, L11.2
- new net N$16: L11.1
- new net N$17: L10.2
- new net N$18: C41.1, L14.2
- new net N$19: L14.1
- new net N$20: L13.2
- new net N$21: C47.1, L17.2
- new net N$22: L17.1
- new net N$23: L16.2
- new net N$24: C49.1, L19.2
- new net N$25: L19.1
- new net N$26: L18.2
- new net N$27: C47.2, C48.2
- new net N$28: C6.1, L21.1, LNA_2.RF_OUT
- new net N$29: C35.2, C36.1
- new net N$30: C2.1, L20.1, LNA_1.RF_OUT
- new net N$31: C8.1, L22.2, LNA_3.RF_OUT
- net +5V3: now also C32.1, C33.1, C38.1, C39.1, C44.1, C45.1, L12.2, L15.2, L20.2, L21.2, L6.2, L7.2, L9.2; no longer C19.1, C2.1, C23.1, C27.1, C6.1, C8.1, LNA_1.RF_OUT, LNA_2.RF_OUT, LNA_3.RF_OUT, LNA_4.RF_OUT, LNA_5.RF_OUT, LNA_6.RF_OUT
- net 1.25M_RF_IN_1: now also SAW_7.INPUT
- net GND: now also C32.2, C33.2, C38.2, C39.2, C44.2, C45.2, LNA_7.GND, LNA_7.GND_1, LNA_8.GND, LNA_8.GND_1, LNA_9.GND, LNA_9.GND_1, X4G$1.GND, X5G$1.GND, X6G$1.GND
Other:
- note added: "1.25m Band"
- note added: "2m Band"
- note added: "70cm Band"
- note added: "This is from DECPU, there is a 5.3V output and this may be compatible, althought it does have a lot of pins that need to be soldered."

Commit message: All components should be connected to ground as well as all pre_pwr wires have been routed. 4 air wires remain...
Parts:
- removed L47: 56n 1206, NewSDR:L-US1206
- removed U$1, U$2, U$3, U$4: TA1914A, SeniorDesign:TA1914A
- added C100, C101, C53, C54, C58, C59, C62, C63, C66, C67, C70, C71, C76, C77, C80, C81, C84, C85, C88, C89, C92, C93, C96, C97: 470n, rcl:C-USC0402K
- added C102, C103, C55, C56, C60, C61, C64, C65, C68, C69, C74, C75, C78, C79, C82, C83, C86, C87, C90, C91, C94, C95, C98, C99: NFM21PS106B0J3D, DEEP EDDY:NFM21PS
- added C50: 160p, rcl:C-USC0603K
- added C51: 180p, rcl:C-USC0603K
- added L23, L24, L25, L26: 100n, NewSDR:L-US1206
- added LDO_1, LDO_10, LDO_11, LDO_12, LDO_2, LDO_3, LDO_4, LDO_5, LDO_6, LDO_7, LDO_8, LDO_9: TPS7A8101DRB, DEEP EDDY:TPS7A8101DRB
- added LNA_10, LNA_11, LNA_12: SPF-5043Z, SeniorDesign:SPF-5043Z
- added R1, R10, R11, R14, R15, R19, R21, R23, R24, R26, R27, R29, R3, R30, R32, R33, R35, R36, R38, R39, R41, R5, R7, R8: 10.0k, rcl:R-US_R0603
- added R12, R16, R2, R22, R25, R28, R31, R34, R37, R40, R6, R9: 52.3k, rcl:R-US_R0603
- added SAW_10, SAW_11, SAW_12, SAW_9: TA1914A, SeniorDesign:TA1914A
- added SAW_13, SAW_14, SAW_15, SAW_16: S511214, SeniorDesign:S511214
- added TP_1, TP_10, TP_11, TP_12, TP_2, TP_3, TP_4, TP_5, TP_6, TP_7, TP_8, TP_9: TPTP20SQ, testpad:TPTP20SQ
- added X10, X11, X12, X13, X14, X15, X16, X17, X18, X19, X20, X21, X22, X23, X24, X25, X26, X27, X28, X29, X30, X31, X32, X7, X8, X9: 0733660061, con-coax:BU-SMA-V
- C1, C11, C18, C20, C22, C24, C26, C28, C3, C30, C32, C36, C37: value 100p 50v c0g -> 100p
- C10: value 0.1u 16V X7R -> 0.1u
- C12, C8: value 100p 50v c0g -> 8p
- C13: value 0.1u 16V X7R -> 12p
- C14, C16: value 8p 5% 0603 -> 100p
- C15: value 12p 5% 0603 -> 0.1u
- C17, C7: value 12p 5% 0603 -> 100p
- C19, C2, C23, C27, C31, C44: value 100p 50v c0g -> 0.1u
- C21, C25, C29, C33, C45: value 0.1u 16V X7R -> 100p
- C34, C41, C49: value 2pF -> 100p
- C35, C40, C48: value 2pF -> 0.1u
- C38, C42: value 100p 50v c0g -> 160p
- C39: value 0.1u 16V X7R -> 180p
- C4: value 0.1u 16V X7R -> 8p
- C43: value 100p 50v c0g -> 180p
- C46: value 2pF -> 160p
- C47: value 2pF -> 180p
- C5, C9: value 100p 50v c0g -> 12p
- C6: value 8p 5% 0603 -> 0.1u
- L1: value 47n 1206 -> 100n
- L10, L13, L16, L18: value 86n 1206 -> 100n
- L11, L14, L17, L19: value 84n 1206 -> 100n
- L12, L15, L20, L21, L22, L7: value 100n 1206 -> 100n
- L2: value 56n 1206 -> 56n
- L3: value 47n 1206 -> 47n
- L4: value 56n 1206 -> 100n
- L5: value 47n 1206 -> 56n
- L6, L9: value 100n 1206 -> 47n
- L8: value 100n 1206 -> 56n
- TP10: value TPSQTP20SQD -> TPSQB1,27; device testpad:TPSQTP20SQD -> testpad:TPSQB1,27
Connections:
- net N$1 renamed LNA_2_IN
- removed net 1.25M_RF_IN1: C26.2, LNA_6.RF_IN
- removed net 1.25M_RF_IN2: C31.2, C34.2
- removed net 1.25M_RF_IN3: C22.1, C22.2, LNA_5.RF_IN, SAW_5.OUTPUT
- removed net 1.25M_RF_IN4: C37.2, C40.2
- removed net 1.25M_RF_IN5: C43.2, C46.2
- removed net 1.25M_RF_IN_: C23.2, SAW_6.INPUT
- removed net 1.25M_RF_IN_1: C27.2, SAW_7.INPUT
- removed net 1.2M5_RF_IN4: C26.1, SAW_6.OUTPUT
- removed net 2M_RF_IN1: X2G$1.1
- removed net 2M_RF_IN10: C48.1, L18.1
- removed net 2M_RF_IN11: C49.2, X6G$1.1
- removed net 2M_RF_IN2: C18.1, C18.2, LNA_4.RF_IN, X3G$1.1
- removed net 2M_RF_IN3: SAW_8.OUTPUT, X4G$1.1
- removed net 2M_RF_IN4: C30.1, C30.2, LNA_7.RF_IN, X5G$1.1
- removed net 2M_RF_IN5: C34.1, L10.1
- removed net 2M_RF_IN6: C36.2, LNA_8.RF_IN
- removed net 2M_RF_IN7: C40.1, L13.1
- removed net 2M_RF_IN8: C41.2, C42.1, C42.2, LNA_9.RF_IN
- removed net 2M_RF_IN9: C46.1, L16.1
- removed net GND1: C23.1, L6.1, LNA_5.RF_OUT
- removed net GND2: C19.1, L7.1, LNA_4.RF_OUT
- removed net GND3: L8.1
- removed net GND4: C31.1, L9.1, LNA_7.RF_OUT
- removed net GND5: C37.1, L12.1, LNA_8.RF_OUT
- removed net GND6: C43.1, L15.1, LNA_9.RF_OUT
- removed net N$10: C15.2, C16.1
- removed net N$11: C16.2, L4.2, SAW_4.INPUT
- removed net N$2: C6.2, L47.2, SAW_2.INPUT
- removed net N$21: C47.1, L17.2
- removed net N$23: L16.2
- removed net N$26: L18.2
- removed net N$29: C35.2, C36.1
- removed net N$3: C14.2, L2.2, SAW_3.INPUT
- removed net N$31: C8.1, L22.2, LNA_3.RF_OUT
- removed net N$4: C14.1, C8.2
- removed net N$5: C7.1, L1.2, SAW_2.OUTPUT
- removed net N$6: C11.2, LNA_3.RF_IN
- removed net N$7: SAW_2.CASE_GND, SAW_2.CASE_GND_1, SAW_2.GND, SAW_2.GND_1, SAW_2.GND_2, SAW_2.GND_3
- removed net N$8: C7.2
- removed net N$9: C15.1, L3.2, SAW_3.OUTPUT
- new net 1.25_RF_OUT: SAW_8.OUTPUT, X16G$1.1
- new net 2M_RF_OUT: C13.2, X8G$1.1
- new net 4M_RF_IN: C38.1, L16.1, X25G$1.1
- new net 4M_RF_OUT: C51.2, L26.1, X32G$1.1
- new net 70CM_RF_IN: C26.1, X17G$1.1
- new net 70CM_RF_OUT: SAW_12.OUTPUT, X24G$1.1
- new net LDO_10_5V: C40.1, C41.1, C93.2, C95.OUT, L18.2, R34.1, TP_10.TP
- new net LDO_11_5V: C44.1, C45.1, C97.2, C99.OUT, L21.2, R37.1, TP_11.TP
- new net LDO_12_5V: C101.2, C103.OUT, C48.1, C49.1, L24.2, R40.1, TP_12.TP
- new net LDO_1_5V: C2.1, C3.1, C54.2, C56.OUT, L1.2, R2.1, TP_1.TP
- new net LDO_2_5V: C59.2, C6.1, C61.OUT, C7.1, L4.2, R6.1, TP_2.TP
- new net LDO_3_5V: C10.1, C11.1, C63.2, C65.OUT, L7.1, R9.1, TP_3.TP
- new net LDO_4_5V: C15.1, C16.1, C67.2, C69.OUT, L10.2, R12.1, TP_4.TP
- new net LDO_5_5V: C19.1, C20.1, C71.2, C75.OUT, L11.2, R16.1, TP_5.TP
- new net LDO_6_5V: C23.1, C24.1, C77.2, C79.OUT, L12.1, R22.1, TP_6.TP
- new net LDO_7_5V: C27.1, C28.1, C81.2, C83.OUT, L13.2, R25.1, TP_7.TP
- new net LDO_8_5V: C31.1, C32.1, C85.2, C87.OUT, L14.2, R28.1, TP_8.TP
- new net LDO_9_5V: C35.1, C36.1, C89.2, C91.OUT, L15.2, R31.1, TP_9.TP
- new net LNA_10_IN: C39.2, L17.1, LNA_10.RF_IN
- new net LNA_10_OUT: C42.1, L18.1, L19.1, LNA_10.RF_OUT
- new net LNA_11_IN: C43.2, L20.1, LNA_11.RF_IN
- new net LNA_11_OUT: C46.1, L21.1, L22.1, LNA_11.RF_OUT
- new net LNA_12_IN: C47.2, L23.1, LNA_12.RF_IN
- new net LNA_12_OUT: C50.1, L24.1, L25.1, LNA_12.RF_OUT
- new net LNA_1_IN: C1.2, LNA_1.RF_IN
- new net LNA_1_OUT: C4.1, L1.1, LNA_1.RF_OUT
- new net LNA_2_OUT: C8.2, L4.1, LNA_2.RF_OUT
- new net LNA_3_IN: C9.2, LNA_3.RF_IN
- new net LNA_3_OUT: C12.1, L7.2, LNA_3.RF_OUT
- new net LNA_4_IN: C14.2, LNA_4.RF_IN
- new net LNA_4_OUT: C17.1, L10.1, LNA_4.RF_OUT
- new net LNA_5_IN: C18.2, LNA_5.RF_IN
- new net LNA_5_OUT: C21.1, L11.1, LNA_5.RF_OUT
- new net LNA_6_IN: C22.2, LNA_6.RF_IN
- new net LNA_6_OUT: C25.1, L12.2, LNA_6.RF_OUT
- new net LNA_7_IN: C26.2, LNA_7.RF_IN
- new net LNA_7_OUT: C29.1, L13.1, LNA_7.RF_OUT
- new net LNA_8_IN: C30.2, LNA_8.RF_IN
- new net LNA_8_OUT: C33.1, L14.1, LNA_8.RF_OUT
- new net LNA_9_IN: C34.2, LNA_9.RF_IN
- new net LNA_9_OUT: C37.1, L15.1, LNA_9.RF_OUT
- new net N$33: C69.IN, LDO_4.OUT
- new net N$34: C71.1, LDO_5.FB/SNS, R16.2, R19.1
- new net N$36: C70.1, LDO_5.NR
- new net N$38: C74.OUT, LDO_5.IN
- new net N$39: C75.IN, LDO_5.OUT
- new net N$40: C81.1, LDO_7.FB/SNS, R25.2, R26.1
- new net N$41: C77.1, LDO_6.FB/SNS, R22.2, R23.1
- new net N$42: C76.1, LDO_6.NR
- new net N$43: C78.OUT, LDO_6.IN
- new net N$45: C79.IN, LDO_6.OUT
- new net N$46: C80.1, LDO_7.NR
- new net N$47: C82.OUT, LDO_7.IN
- new net N$48: C83.IN, LDO_7.OUT
- new net N$49: C85.1, LDO_8.FB/SNS, R28.2, R29.1
- new net N$50: C84.1, LDO_8.NR
- new net N$51: C86.OUT, LDO_8.IN
- new net N$52: C87.IN, LDO_8.OUT
- new net N$53: C89.1, LDO_9.FB/SNS, R31.2, R32.1
- new net N$54: C88.1, LDO_9.NR
- new net N$56: C90.OUT, LDO_9.IN
- new net N$57: C91.IN, LDO_9.OUT
- new net N$61: C93.1, LDO_10.FB/SNS, R34.2, R35.1
- new net N$62: C92.1, LDO_10.NR
- new net N$63: C94.OUT, LDO_10.IN
- new net N$64: C95.IN, LDO_10.OUT
- new net N$66: C97.1, LDO_11.FB/SNS, R37.2, R38.1
- new net N$67: C96.1, LDO_11.NR
- new net N$68: C98.OUT, LDO_11.IN
- new net N$69: C99.IN, LDO_11.OUT
- new net N$70: C101.1, LDO_12.FB/SNS, R40.2, R41.1
- new net N$71: C100.1, LDO_12.NR
- new net N$72: C102.OUT, LDO_12.IN
- new net N$73: C103.IN, LDO_12.OUT
- new net PRE_PWR_10: LDO_1.EN, LDO_10.EN, LDO_11.EN, LDO_2.EN, LDO_3.EN, LDO_4.EN, LDO_5.EN, LDO_6.EN, LDO_7.EN, LDO_8.EN, LDO_9.EN, R1.2, R11.2, R15.2, R21.2, R24.2, R27.2, R30.2, R33.2, R36.2, R5.2, R8.2
- new net PRE_PWR_12: LDO_12.EN, R39.2
- new net SAW+6_OUT: C22.1, SAW_6.OUTPUT, X13G$1.1
- new net SAW_10_IN: C33.2, SAW_10.INPUT, X20G$1.1
- new net SAW_10_OUT: C34.1, SAW_10.OUTPUT, X21G$1.1
- new net SAW_11_12_RF: SAW_11.OUTPUT, SAW_12.INPUT, X23G$1.1
- new net SAW_11_IN: C37.2, SAW_11.INPUT, X22G$1.1
- new net SAW_13_IN: C38.2, SAW_13.INPUT
- new net SAW_13_OUT: C39.1, SAW_13.OUTPUT, X26G$1.1
- new net SAW_14_IN: C42.2, SAW_14.INPUT, X27G$1.1
- new net SAW_14_OUT: C43.1, SAW_14.OUTPUT, X28G$1.1
- new net SAW_15_IN: C46.2, SAW_15.INPUT, X29G$1.1
- new net SAW_15_OUT: C47.1, SAW_15.OUTPUT, X30G$1.1
- new net SAW_16_IN: C50.2, SAW_16.INPUT, X31G$1.1
- new net SAW_16_OUT: C51.1, SAW_16.OUTPUT
- new net SAW_1_OUT: C1.1, SAW_1.OUTPUT, X2G$1.1
- new net SAW_2_IN: C4.2, L2.2, SAW_2.INPUT, X3G$1.1
- new net SAW_2_OUT: C5.1, L3.2, SAW_2.OUTPUT, X4G$1.1
- new net SAW_3_IN: C8.1, L5.2, SAW_3.INPUT, X5G$1.1
- new net SAW_3_OUT: C9.1, L6.2, SAW_3.OUTPUT, X6G$1.1
- new net SAW_4_IN: C12.2, L8.2, SAW_4.INPUT, X7G$1.1
- new net SAW_4_OUT: C13.1, L9.2, SAW_4.OUTPUT
- new net SAW_5_IN: C17.2, SAW_5.INPUT, X10G$1.1
- new net SAW_5_OUT: C18.1, SAW_5.OUTPUT, X11G$1.1
- new net SAW_6_IN: C21.2, SAW_6.INPUT, X12G$1.1
- new net SAW_7_8_RF: SAW_7.OUTPUT, SAW_8.INPUT, X15G$1.1
- new net SAW_7_IN: C25.2, SAW_7.INPUT, X14G$1.1
- new net SAW_9_IN: C29.2, SAW_9.INPUT, X18G$1.1
- new net SAW_9_OUT: C30.1, SAW_9.OUTPUT, X19G$1.1
- net +5V3: now also C102.IN, C55.IN, C60.IN, C64.IN, C68.IN, C74.IN, C78.IN, C82.IN, C86.IN, C90.IN, C94.IN, C98.IN, R1.1, R11.1, R15.1, R21.1, R24.1, R27.1, R30.1, R33.1, R36.1, R39.1, R5.1, R8.1; no longer C10.1, C12.1, C13.1, C20.1, C21.1, C24.1, C25.1, C28.1, C29.1, C3.1, C32.1, C33.1, C38.1, C39.1, C4.1, C44.1, C45.1, C9.1, L12.2, L15.2, L20.2, L21.2, L6.2, L7.2, L9.2
- net 1.25M_RF_IN: now also C14.1, X9G$1.1; no longer C19.2, SAW_5.INPUT
- net 2M_RF_IN: no longer C1.1, C1.2, C2.2, C5.1, LNA_1.RF_IN, SAW_1.OUTPUT
- net GND: now also C100.2, C102.GND, C103.GND, C11.2, C15.2, C16.2, C19.2, C2.2, C23.2, C27.2, C31.2, C35.2, C36.2, C40.2, C41.2, C48.2, C49.2, C53.2, C55.GND, C56.GND, C58.2, C6.2, C60.GND, C61.GND, C62.2, C64.GND, C65.GND, C66.2, C68.GND, C69.GND, C7.2, C70.2, C74.GND, C75.GND, C76.2, C78.GND, C79.GND, C80.2, C82.GND, C83.GND, C84.2, C86.GND, C87.GND, C88.2, C90.GND, C91.GND, C92.2, C94.GND, C95.GND, C96.2, C98.GND, C99.GND, L16.2, L17.2, L19.2, L20.2, L22.2, L23.2, L25.2, L26.2, L6.1, L8.1, L9.1, LDO_1.GND, LDO_10.GND, LDO_11.GND, LDO_12.GND, LDO_2.GND, LDO_3.GND, LDO_4.GND, LDO_5.GND, LDO_6.GND, LDO_7.GND, LDO_8.GND, LDO_9.GND, LNA_10.GND, LNA_10.GND_1, LNA_11.GND, LNA_11.GND_1, LNA_12.GND, LNA_12.GND_1, R10.2, R14.2, R19.2, R23.2, R26.2, R29.2, R3.2, R32.2, R35.2, R38.2, R41.2, R7.2, SAW_10.GND, SAW_10.GND_1, SAW_10.GND_2, SAW_10.GND_3, SAW_11.GND, SAW_11.GND_1, SAW_11.GND_2, SAW_11.GND_3, SAW_12.GND, SAW_12.GND_1, SAW_12.GND_2, SAW_12.GND_3, SAW_13.GROUND_1, SAW_13.GROUND_2, SAW_13.GROUND_3, SAW_13.GROUND_4, SAW_13.GROUND_5, SAW_13.GROUND_6, SAW_13.INPUT_GROUND, SAW_13.OUTPUT_GROUND, SAW_14.GROUND_1, SAW_14.GROUND_2, SAW_14.GROUND_3, SAW_14.GROUND_4, SAW_14.GROUND_5, SAW_14.GROUND_6, SAW_14.INPUT_GROUND, SAW_14.OUTPUT_GROUND, SAW_15.GROUND_1, SAW_15.GROUND_2, SAW_15.GROUND_3, SAW_15.GROUND_4, SAW_15.GROUND_5, SAW_15.GROUND_6, SAW_15.INPUT_GROUND, SAW_15.OUTPUT_GROUND, SAW_16.GROUND_1, SAW_16.GROUND_2, SAW_16.GROUND_3, SAW_16.GROUND_4, SAW_16.GROUND_5, SAW_16.GROUND_6, SAW_16.INPUT_GROUND, SAW_16.OUTPUT_GROUND, SAW_2.CASE_GND, SAW_2.CASE_GND_1, SAW_2.GND, SAW_2.GND_1, SAW_2.GND_2, SAW_2.GND_3, SAW_5.CASE_GND, SAW_5.CASE_GND_1, SAW_5.GND, SAW_5.GND_1, SAW_5.GND_2, SAW_5.GND_3, SAW_6.CASE_GND, SAW_6.CASE_GND_1, SAW_6.GND, SAW_6.GND_1, SAW_6.GND_2, SAW_6.GND_3, SAW_7.CASE_GND, SAW_7.CASE_GND_1, SAW_7.GND, SAW_7.GND_1, SAW_7.GND_2, SAW_7.GND_3, SAW_8.CASE_GND, SAW_8.CASE_GND_1, SAW_8.GND, SAW_8.GND_1, SAW_8.GND_2, SAW_8.GND_3, SAW_9.GND, SAW_9.GND_1, SAW_9.GND_2, SAW_9.GND_3, X10G$1.GND, X11G$1.GND, X12G$1.GND, X13G$1.GND, X14G$1.GND, X15G$1.GND, X16G$1.GND, X17G$1.GND, X18G$1.GND, X19G$1.GND, X20G$1.GND, X21G$1.GND, X22G$1.GND, X23G$1.GND, X24G$1.GND, X25G$1.GND, X26G$1.GND, X27G$1.GND, X28G$1.GND, X29G$1.GND, X30G$1.GND, X31G$1.GND, X32G$1.GND, X7G$1.GND, X8G$1.GND, X9G$1.GND; no longer C12.2, C13.2, C21.2, C25.2, C29.2, C33.2, C38.2, C39.2, C4.2, C9.2, L1.1, L4.1, L47.1
- net N$12: now also C54.1, LDO_1.FB/SNS, R2.2, R3.1; no longer C17.1, L5.2, SAW_4.OUTPUT
- net N$13: now also C53.1, LDO_1.NR; no longer C27.1, L8.2, LNA_6.RF_OUT
- net N$14: now also C55.OUT, LDO_1.IN; no longer SAW_7.OUTPUT, SAW_8.INPUT
- net N$15: now also C56.IN, LDO_1.OUT; no longer C35.1, L11.2
- net N$16: now also C59.1, LDO_2.FB/SNS, R6.2, R7.1; no longer L11.1
- net N$17: now also C58.1, LDO_2.NR; no longer L10.2
- net N$18: now also C60.OUT, LDO_2.IN; no longer C41.1, L14.2
- net N$19: now also C61.IN, LDO_2.OUT; no longer L14.1
- net N$20: now also C63.1, LDO_3.FB/SNS, R10.1, R9.2; no longer L13.2
- net N$22: now also C62.1, LDO_3.NR; no longer L17.1
- net N$24: now also C64.OUT, LDO_3.IN; no longer C49.1, L19.2
- net N$25: now also C65.IN, LDO_3.OUT; no longer L19.1
- net N$27: now also C67.1, LDO_4.FB/SNS, R12.2, R14.1; no longer C47.2, C48.2
- net N$28: now also C66.1, LDO_4.NR; no longer C6.1, L21.1, LNA_2.RF_OUT
- net N$30: now also C68.OUT, LDO_4.IN; no longer C2.1, L20.1, LNA_1.RF_OUT
Other:
- note added: "+5V"
- note added: "ENABLE PRE_PWR FOR BITE1"
- note added: "REV B HAD PCHAN FET HERE GROUND GATE"
